File: MAG Synth/Stylish-Belt-Synth - Full.kicad_pcb (KiCad board)
At the start: 2 copper layers, 177.8 x 101.7 mm, 63 parts, among them J0 USB_B, J1 Audio-Jack-3_2Switches, J26 WRITE PATCH, J27 PARAM SELECT, J28 PATCH SELECT, J29 MODE, J30 STYLUS, SW1 Power, U1 stm32f103c8t6-module-china, U2 XPT8871

Commit message: Latest
Parts:
- added REF**: 1pin, Connect:1pin, F.Cu at (74.2, 60.8)
- added REF**: 1pin, Connect:1pin, F.Cu at (222.3, 60.8)
- added REF**: 1pin, Connect:1pin, F.Cu at (222.3, 149.4)
- added REF**: 1pin, Connect:1pin, F.Cu at (74.2, 149.4)
- CA1: footprint SoftEggKiCAD:C_Disc_D5.0mm_W2.5mm_P5.00mm+SMD -> Capacitors_ThroughHole:CP_Radial_Tantal_D4.5mm_P2.50mm
- CA3: footprint Capacitors_ThroughHole:CP_Radial_Tantal_D4.5mm_P2.50mm -> SoftEggKiCAD:C_Disc_D5.0mm_W2.5mm_P5.00mm+SMD
- LS1: value Speaker -> SPEAKER
- moved J1 6.71 mm to (213.2, 62.9), turned to 250 degrees
- moved CA3 4.33 mm to (189.9, 92.7), turned to 270 degrees
- moved LS1 3.70 mm to (197.6, 61.4)
Routing:
- net /+5V: track 337.9 -> 360.0 mm, vias 18 -> 20
- net Net-(J1-Pad4): track 63.9 -> 52.6 mm
- net /XH-M125-amp-board/OUT-: track 92.5 -> 84.7 mm
- net /XH-M125-amp-board/OUT+: track 108.6 -> 104.1 mm
- net /E1: track 43.4 -> 46.8 mm
- net /F1: track 48.3 -> 51.3 mm
- net GND: track 536.6 -> 534.1 mm
- net /G1: track 73.0 -> 75.1 mm
- net /A#1: track 90.9 -> 92.7 mm
- net /C2: track 115.1 -> 116.5 mm
- net /PARAM: track 141.8 -> 142.8 mm
- net /G0: track 146.7 -> 147.7 mm
Other:
- outline, holes or cut-outs redrawn
- net class Default: trace_width 0.508 -> 0.2
- board text added: "+"
- board text added: "."

Commit message: Updated PCB to have contiguous outline. Yet another incomplete reworking of the state machine.
Routing:
- net GND: track 534.1 -> 549.0 mm, vias 16 -> 17
- net Net-(C1-Pad2): track 3.23 -> 10.0 mm
- net /+5V: track 360.0 -> 364.2 mm, vias 20 -> 21
- net Net-(CA4-Pad1): track 4.48 -> 7.55 mm
- net /AUDIO_OUT: track 56.7 -> 58.4 mm
- net Net-(R3-Pad1): track 10.0 -> 11.7 mm
- net /A#1: track 92.7 -> 93.8 mm
Other:
- outline, holes or cut-outs redrawn
