File: MAG Synth/WS2812B-16-LED-RING.sch (KiCad schematic (older format))
At the start: 33 parts

Commit message: New power switch. 3d model included. 3d model of the amp board included. PCB redesign in progress.
Parts:
- CL0, CL1, CL10, CL11, CL12, CL13, CL14, CL15, CL2, CL3, CL4, CL5, CL6, CL7, CL8, CL9: footprint (none) -> Capacitors_SMD:C_0805_HandSoldering
- RGB0: renamed from D0; footprint WS2812B -> WS2812B:WS2812B
- RGB1: renamed from D1; footprint WS2812B -> WS2812B:WS2812B
- RGB10: renamed from D10; footprint WS2812B -> WS2812B:WS2812B
- RGB11: renamed from D11; footprint WS2812B -> WS2812B:WS2812B
- RGB12: renamed from D12; footprint WS2812B -> WS2812B:WS2812B
- RGB13: renamed from D13; footprint WS2812B -> WS2812B:WS2812B
- RGB14: renamed from D14; footprint WS2812B -> WS2812B:WS2812B
- RGB15: renamed from D15; footprint WS2812B -> WS2812B:WS2812B
- RGB2: renamed from D2; footprint WS2812B -> WS2812B:WS2812B
- RGB3: renamed from D3; footprint WS2812B -> WS2812B:WS2812B
- RGB4: renamed from D4; footprint WS2812B -> WS2812B:WS2812B
- RGB5: renamed from D5; footprint WS2812B -> WS2812B:WS2812B
- RGB6: renamed from D6; footprint WS2812B -> WS2812B:WS2812B
- RGB7: renamed from D7; footprint WS2812B -> WS2812B:WS2812B
- RGB8: renamed from D8; footprint WS2812B -> WS2812B:WS2812B
- RGB9: renamed from D9; footprint WS2812B -> WS2812B:WS2812B
- renumbered J2 to JL1

Commit message: V3 board V2.4 case
Connections:
- net 5V renamed VIN
Changed lines of the file:
@@
-EESchema Schematic File Version 4
+EESchema Schematic File Version 5
 LIBS:Stylish-Belt-Synth - Full-cache
-EELAYER 28 0
+EELAYER 29 0
 EELAYER END
 $Descr A4 11693 8268
 encoding utf-8
-Sheet 3 3
-Title ""
-Date ""
-Rev ""
+Sheet 2 2
+Title "\"Stylish\" Trucker Belt Stylus Synthesizer"
+Date "2019-05-07"
+Rev "0.3"
 Comp "SoftEgg"
 Comment1 "V0.1 T.B. Trzepacz 2018/2/19"
 Comment2 "V0.2 T.B. Trzepacz 2018/10/14"
-Comment3 ""
+Comment3 "V0.3 T.B Trzepacz 2019/5/7"
 Comment4 ""
 $EndDescr
@@
 DIN
 Text HLabel 3100 750  0    50   Input ~ 0
-5V
+VIN
 Text HLabel 4500 600  2    50   Input ~ 0
 DOUT
