File: MAG Synth/XH-M125-amp-board.sch (KiCad schematic (older format))
At the start: 7 parts, among them J1 Conn_01x06, U2 XPT8871

Commit message: New power switch. 3d model included. 3d model of the amp board included. PCB redesign in progress.
Parts:
- CA3: footprint Capacitors_SMD:C_0805_HandSoldering -> Capacitors_ThroughHole:CP_Radial_Tantal_D4.5mm_P2.50mm
- renumbered J1 to JA1
Changed lines of the file:
@@
 EESchema Schematic File Version 4
 LIBS:Stylish-Belt-Synth - Full-cache
-EELAYER 26 0
+EELAYER 28 0
 EELAYER END
 $Descr A4 11693 8268
@@
 Rev "1"
 Comp "SoftEgg"
-Comment1 "V1.0 T.B. Trzepacz 2018/2/19"
-Comment2 ""
+Comment1 "V0.1 T.B. Trzepacz 2018/2/19"
+Comment2 "V0.2 T.B. Trzepacz 2018/10/14"
 Comment3 ""
 Comment4 ""
@@
 F 0 "CA3" V 5725 3625 50  0000 L CNN
 F 1 "1uF" V 5525 3625 50  0000 L CNN
-F 2 "Capacitors_SMD:C_0805_HandSoldering" H 5625 3675 50  0001 C CNN
+F 2 "Capacitors_ThroughHole:CP_Radial_Tantal_D4.5mm_P2.50mm" H 5625 3675 50  0001 C CNN
 F 3 "" H 5625 3675 50  0001 C CNN
 	1    5625 3675
@@
 	5525 4200 5525 4275
 $Comp
-L conn:Conn_01x06 J1
+L conn:Conn_01x06 JA1
 U 1 1 5AA56D62
 P 3575 3675
-F 0 "J1" H 3495 4092 50  0000 C CNN
+F 0 "JA1" H 3495 4092 50  0000 C CNN
 F 1 "Conn_01x06" H 3495 4001 50  0000 C CNN
 F 2 "Pin_Headers:Pin_Header_Straight_1x06_Pitch2.54mm" H 3575 3675 50  0001 C CNN

Commit message: Updated footprints. Including STL for speaker holder.
Parts:
- CA1: value 470uF -> 470μF; footprint Capacitors_SMD:C_0805_HandSoldering -> SoftEggKiCAD:C_Disc_D5.0mm_W2.5mm_P5.00mm+SMD
- CA2: value 1uF -> 1μF; footprint Capacitors_SMD:C_0805_HandSoldering -> SoftEggKiCAD:C_Disc_D5.0mm_W2.5mm_P5.00mm+SMD
- CA3: value 1uF -> 1μF
- CA4: value 0.39uF -> 0.39μF; footprint Capacitors_SMD:C_0805_HandSoldering -> SoftEggKiCAD:C_Disc_D5.0mm_W2.5mm_P5.00mm+SMD
- R3: value R -> 100Ω; footprint Resistors_SMD:R_0805_HandSoldering -> SoftEggKiCAD:R_Axial_DIN0204_L3.6mm_D1.6mm_P7.62mm_Horizontal+SMD804
Changed lines of the file:
@@
 P 5625 4275
 F 0 "CA2" V 5675 4125 50  0000 L CNN
-F 1 "1uF" V 5675 4325 50  0000 L CNN
-F 2 "Capacitors_SMD:C_0805_HandSoldering" H 5625 4275 50  0001 C CNN
+F 1 "1μF" V 5675 4325 50  0000 L CNN
+F 2 "SoftEggKiCAD:C_Disc_D5.0mm_W2.5mm_P5.00mm+SMD" H 5625 4275 50  0001 C CNN
 F 3 "" H 5625 4275 50  0001 C CNN
 	1    5625 4275
@@
 P 5625 4125
 F 0 "CA1" V 5550 3975 50  0000 L CNN
-F 1 "470uF" V 5550 4175 50  0000 L CNN
-F 2 "Capacitors_SMD:C_0805_HandSoldering" H 5625 4125 50  0001 C CNN
+F 1 "470μF" V 5550 4175 50  0000 L CNN
+F 2 "SoftEggKiCAD:C_Disc_D5.0mm_W2.5mm_P5.00mm+SMD" H 5625 4125 50  0001 C CNN
 F 3 "" H 5625 4125 50  0001 C CNN
 	1    5625 4125
@@
 P 5575 3275
 F 0 "R3" V 5475 3275 50  0000 C CNN
-F 1 "R" V 5575 3275 50  0000 C CNN
-F 2 "Resistors_SMD:R_0805_HandSoldering" V 5505 3275 50  0001 C CNN
+F 1 "100Ω" V 5575 3275 50  0000 C CNN
+F 2 "SoftEggKiCAD:R_Axial_DIN0204_L3.6mm_D1.6mm_P7.62mm_Horizontal+SMD804" V 5505 3275 50  0001 C CNN
 F 3 "" H 5575 3275 50  0001 C CNN
 	1    5575 3275
@@
 P 5250 3275
 F 0 "CA4" V 5150 3225 50  0000 L CNN
-F 1 "0.39uF" V 5350 3175 50  0000 L CNN
-F 2 "Capacitors_SMD:C_0805_HandSoldering" H 5250 3275 50  0001 C CNN
+F 1 "0.39μF" V 5350 3175 50  0000 L CNN
+F 2 "SoftEggKiCAD:C_Disc_D5.0mm_W2.5mm_P5.00mm+SMD" H 5250 3275 50  0001 C CNN
 F 3 "" H 5250 3275 50  0001 C CNN
 	1    5250 3275
@@
 P 5625 3675
 F 0 "CA3" V 5725 3625 50  0000 L CNN
-F 1 "1uF" V 5525 3625 50  0000 L CNN
+F 1 "1μF" V 5525 3625 50  0000 L CNN
 F 2 "Capacitors_ThroughHole:CP_Radial_Tantal_D4.5mm_P2.50mm" H 5625 3675 50  0001 C CNN
 F 3 "" H 5625 3675 50  0001 C CNN
