File: MAG Synth/Stylish-Belt-Synth - Full.sch (KiCad schematic (older format))
At the start: 17 parts, among them J26 WRITE PATCH, J27 PARAM SELECT, J28 PATCH SELECT, J29 MODE, J30 STYLUS, SW1 Power, U1 stm32f103c8t6-module-china

Commit message: Schematic updated with USB and diodes for MODE button. Source code updated with state machine in process.
Parts:
- added D1, D2: 1N4148, Diodes_ThroughHole:D_DO-35_SOD27_P7.62mm_Horizontal, symbol diode:1N4148
- added D1B, D2B: 1N4148, Diodes_SMD:D_0805, symbol diode:1N4148
- added J0: USB_B, Connectors:USB_B, symbol conn:USB_B
- R1B: renamed from R4; footprint Resistors_ThroughHole:R_Axial_DIN0207_L6.3mm_D2.5mm_P2.54mm_Vertical -> Resistors_ThroughHole:R_Axial_DIN0204_L3.6mm_D1.6mm_P7.62mm_Horizontal
- R2B: renamed from R5; footprint Resistors_ThroughHole:R_Axial_DIN0207_L6.3mm_D2.5mm_P2.54mm_Vertical -> Resistors_ThroughHole:R_Axial_DIN0207_L6.3mm_D2.5mm_P7.62mm_Horizontal
- renumbered C2 to C1B
Connections:
- net labels removed: MODE
- wire segments 39 -> 60
Other:
- moved on the sheet: J26, J27, J28
Changed lines of the file:
@@
 L conn:Conn_01x01_Male J28
 U 1 1 5A85684E
-P 9075 3200
-F 0 "J28" H 8975 3200 50  0000 C CNN
-F 1 "PATCH SELECT" H 8900 3200 50  0000 R CNN
-F 2 "SoftEggKiCAD:LargeRoundTouchPad" H 9075 3200 50  0001 C CNN
-F 3 "" H 9075 3200 50  0001 C CNN
-	1    9075 3200
+P 9075 2675
+F 0 "J28" H 8975 2675 50  0000 C CNN
+F 1 "PATCH SELECT" H 8900 2675 50  0000 R CNN
+F 2 "SoftEggKiCAD:LargeRoundTouchPad" H 9075 2675 50  0001 C CNN
+F 3 "" H 9075 2675 50  0001 C CNN
+	1    9075 2675
 	-1   0    0    1
 $EndComp
@@
 L conn:Conn_01x01_Male J27
 U 1 1 5A856A96
-P 9075 3050
-F 0 "J27" H 8975 3050 50  0000 C CNN
-F 1 "PARAM SELECT" H 8900 3050 50  0000 R CNN
-F 2 "SoftEggKiCAD:LargeRoundTouchPad" H 9075 3050 50  0001 C CNN
-F 3 "" H 9075 3050 50  0001 C CNN
-	1    9075 3050
+P 9075 3025
+F 0 "J27" H 8975 3025 50  0000 C CNN
+F 1 "PARAM SELECT" H 8900 3025 50  0000 R CNN
+F 2 "SoftEggKiCAD:LargeRoundTouchPad" H 9075 3025 50  0001 C CNN
+F 3 "" H 9075 3025 50  0001 C CNN
+	1    9075 3025
 	-1   0    0    1
 $EndComp
@@
 L conn:Conn_01x01_Male J26
 U 1 1 5A856E54
-P 9075 2900
-F 0 "J26" H 8975 2900 50  0000 C CNN
-F 1 "WRITE PATCH" H 8900 2900 50  0000 R CNN
-F 2 "SoftEggKiCAD:LargeRoundTouchPad" H 9075 2900 50  0001 C CNN
-F 3 "" H 9075 2900 50  0001 C CNN
-	1    9075 2900
+P 9075 2850
+F 0 "J26" H 8975 2850 50  0000 C CNN
+F 1 "WRITE PATCH" H 8900 2850 50  0000 R CNN
+F 2 "SoftEggKiCAD:LargeRoundTouchPad" H 9075 2850 50  0001 C CNN
+F 3 "" H 9075 2850 50  0001 C CNN
+	1    9075 2850
 	-1   0    0    1
 $EndComp
@@
 U 1 1 5A8BA68B
 P 8450 5875
-F 0 "C1" V 8550 5775 50  0000 L CNN
+F 0 "C1" V 8350 5850 50  0000 L CNN
 F 1 "1uF" H 8460 5795 50  0001 L CNN
 F 2 "Capacitors_SMD:C_0805_HandSoldering" H 8450 5875 50  0001 C CNN
@@
 	10650 6200 7525 6200
 Wire Notes Line
-	8525 2800 9850 2800
-Wire Notes Line
-	9850 2800 9850 3625
-Wire Notes Line
-	9850 3625 8525 3625
-Wire Notes Line
-	8525 3625 8525 2800
+	7775 2600 9850 2600
+Wire Notes Line
+	9850 2600 9850 3625
+Wire Notes Line
+	9850 3625 7775 3625
+Wire Notes Line
+	7775 3625 7775 2600
 Text Notes 8875 3600 0    60   ~ 0
 PCB UI Pads\nfor Stylus
@@
 Connection ~ 1800 5675
 $Comp
-L device:R R4
+L device:R R1B
 U 1 1 5B95BBFA
-P 8200 5950
-F 0 "R4" V 8280 5950 50  0000 C CNN
-F 1 "10k" V 8200 5950 50  0000 C CNN
-F 2 "Resistors_ThroughHole:R_Axial_DIN0207_L6.3mm_D2.5mm_P2.54mm_Vertical" V 8130 5950 50  0001 C CNN
-F 3 "" H 8200 5950 50  0001 C CNN
-	1    8200 5950
+P 8200 5975
+F 0 "R1B" V 8280 5975 50  0001 C CNN
+F 1 "10k" V 8200 5975 50  0000 C CNN
+F 2 "Resistors_ThroughHole:R_Axial_DIN0204_L3.6mm_D1.6mm_P7.62mm_Horizontal" V 8130 5975 50  0001 C CNN
+F 3 "" H 8200 5975 50  0001 C CNN
+	1    8200 5975
 	0    1    1    0
 $EndComp
@@
 	10650 5525 10650 6200
 $Comp
-L device:C_Small C2
+L device:C_Small C1B
 U 1 1 5B9899BC
 P 8600 5875
-F 0 "C2" V 8700 5775 50  0000 L CNN
+F 0 "C1B" V 8700 5775 50  0001 L CNN
 F 1 "1uF" H 8610 5795 50  0001 L CNN
 F 2 "Capacitors_ThroughHole:C_Disc_D5.0mm_W2.5mm_P5.00mm" H 8600 5875 50  0001 C CNN
@@
 $EndComp
 $Comp
-L device:R R5
+L device:R R2B
 U 1 1 5B989A42
 P 9025 5925
-F 0 "R5" V 9105 5925 50  0000 C CNN
+F 0 "R2B" V 9105 5925 50  0001 C CNN
 F 1 "1k" V 9025 5925 50  0000 C CNN
-F 2 "Resistors_ThroughHole:R_Axial_DIN0207_L6.3mm_D2.5mm_P2.54mm_Vertical" V 8955 5925 50  0001 C CNN
+F 2 "Resistors_ThroughHole:R_Axial_DIN0207_L6.3mm_D2.5mm_P7.62mm_Horizontal" V 8955 5925 50  0001 C CNN
 F 3 "" H 9025 5925 50  0001 C CNN
 	1    9025 5925
@@
 $EndComp
 Wire Wire Line
-	8050 5950 8050 6075
+	8050 5975 8050 6075
 Connection ~ 8050 6075
 Wire Wire Line
-	8350 5950 8350 6075
+	8350 5975 8350 6075
 Connection ~ 8350 6075
 Wire Wire Line
@@
 Text Label 4200 2900 2    50   ~ 0
 F#0
-Text Label 4200 3050 2    50   ~ 0
+Text Label 6300 3350 0    50   ~ 0
 G0
-Text Label 4200 3200 2    50   ~ 0
+Text Label 6300 2600 0    50   ~ 0
 G#0
 Text Label 4200 3350 2    50   ~ 0
@@
 Text Label 6300 3500 0    50   ~ 0
 C2
-Text Label 6300 3350 0    50   ~ 0
-MODE
 Text Label 6300 2750 0    50   ~ 0
 PATCH
@@
 Text Label 6300 2900 0    50   ~ 0
 WRITE
-Text Label 8875 2900 2    50   ~ 0
+Text Label 8025 2850 2    50   ~ 0
 WRITE
-Text Label 8875 3050 2    50   ~ 0
+Text Label 8025 3025 2    50   ~ 0
 PARAM
-Text Label 8875 3200 2    50   ~ 0
+Text Label 8025 2675 2    50   ~ 0
 PATCH
-Text Label 8875 3350 2    50   ~ 0
-MODE
 Text Label 6300 3200 0    50   ~ 0
 LED_DIN
@@
 Text Label 4200 2000 2    50   ~ 0
 C0
+$Comp
+L diode:1N4148 D1
+U 1 1 5BBC38EE
+P 8200 3200
+F 0 "D1" V 8250 3350 50  0000 R CNN
+F 1 "1N4148" V 8150 3550 50  0000 R CNN
+F 2 "Diodes_ThroughHole:D_DO-35_SOD27_P7.62mm_Horizontal" H 8200 3025 50  0001 C CNN
+F 3 "http://www.nxp.com/documents/data_sheet/1N4148_1N4448.pdf" H 8200 3200 50  0001 C CNN
+	1    8200 3200
+	0    -1   -1   0
+$EndComp
+Wire Wire Line
+	8875 2850 8200 2850
+Wire Wire Line
+	8200 2850 8200 3050
+Wire Wire Line
+	8800 3350 8875 3350
+Connection ~ 8800 3350
+$Comp
+L diode:1N4148 D2
+U 1 1 5BBC37C5
+P 8800 3200
+F 0 "D2" V 8846 3121 50  0000 R CNN
+F 1 "1N4148" V 8755 3121 50  0000 R CNN
+F 2 "Diodes_ThroughHole:D_DO-35_SOD27_P7.62mm_Horizontal" H 8800 3025 50  0001 C CNN
+F 3 "http://www.nxp.com/documents/data_sheet/1N4148_1N4448.pdf" H 8800 3200 50  0001 C CNN
+	1    8800 3200
+	0    -1   -1   0
+$EndComp
+Wire Wire Line
+	8875 3025 8800 3025
+Wire Wire Line
+	8800 3025 8800 3050
+Wire Wire Line
+	8800 3025 8675 3025
+Connection ~ 8800 3025
+Wire Wire Line
+	8200 2850 8025 2850
+Connection ~ 8200 2850
+Wire Wire Line
+	8875 2675 8025 2675
+$Comp
+L diode:1N4148 D1B
+U 1 1 5BBE4231
+P 8325 3200
+F 0 "D1B" V 8375 3350 50  0001 R CNN
+F 1 "1N4148" V 8275 3550 50  0001 R CNN
+F 2 "Diodes_SMD:D_0805" H 8325 3025 50  0001 C CNN
+F 3 "http://www.nxp.com/documents/data_sheet/1N4148_1N4448.pdf" H 8325 3200 50  0001 C CNN
+	1    8325 3200
+	0    -1   -1   0
+$EndComp
+Wire Wire Line
+	8325 3050 8200 3050
+Connection ~ 8200 3050
+Wire Wire Line
+	8200 3350 8325 3350
+Connection ~ 8325 3350
+$Comp
+L diode:1N4148 D2B
+U 1 1 5BBE6FB8
+P 8675 3200
+F 0 "D2B" V 8721 3121 50  0001 R CNN
+F 1 "1N4148" V 8675 3121 50  0001 R CNN
+F 2 "Diodes_SMD:D_0805" H 8675 3025 50  0001 C CNN
+F 3 "http://www.nxp.com/documents/data_sheet/1N4148_1N4448.pdf" H 8675 3200 50  0001 C CNN
+	1    8675 3200
+	0    -1   -1   0
+$EndComp
+Wire Wire Line
+	8675 3050 8675 3025
+Connection ~ 8675 3025
+Wire Wire Line
+	8675 3025 8025 3025
+Wire Wire Line
+	8675 3350 8800 3350
+Connection ~ 8675 3350
+Wire Wire Line
+	8325 3350 8675 3350
+$Comp
+L conn:USB_B J0
+U 1 1 5BBEB964
+P 2725 3150
+F 0 "J0" H 2495 3048 50  0000 R CNN
+F 1 "USB_B" H 2495 3139 50  0000 R CNN
+F 2 "Connectors:USB_B" H 2875 3100 50  0001 C CNN
+F 3 "" H 2875 3100 50  0001 C CNN
+	1    2725 3150
+	1    0    0    1
+$EndComp
+Wire Wire Line
+	4200 3050 3025 3050
+Wire Wire Line
+	4200 3200 3025 3200
+Wire Wire Line
+	3025 3200 3025 3150
+Wire Wire Line
+	2725 2750 3275 2750
+$Comp
+L power:GND #PWR?
+U 1 1 5BBEFFF4
+P 3275 2750
+F 0 "#PWR?" H 3275 2500 50  0001 C CNN
+F 1 "GND" H 3280 2577 50  0000 C CNN
+F 2 "" H 3275 2750 50  0001 C CNN
+F 3 "" H 3275 2750 50  0001 C CNN
+	1    3275 2750
+	1    0    0    -1
+$EndComp
+Wire Wire Line
+	3025 3350 3250 3350
+Wire Wire Line
+	3250 3350 3250 4550
+Wire Wire Line
+	3250 4550 4200 4550
 $EndSCHEMATC

Commit message: New power switch. 3d model included. 3d model of the amp board included. PCB redesign in progress.
Parts:
- removed C1B: 1uF, Capacitors_ThroughHole:C_Disc_D5.0mm_W2.5mm_P5.00mm, symbol device:C_Small
- removed D1B: 1N4148, Diodes_SMD:D_0805, symbol diode:1N4148
- removed D2: 1N4148, Diodes_ThroughHole:D_DO-35_SOD27_P7.62mm_Horizontal, symbol diode:1N4148
- removed R1B: 10k, Resistors_ThroughHole:R_Axial_DIN0204_L3.6mm_D1.6mm_P7.62mm_Horizontal, symbol device:R
- removed R2B: 1k, Resistors_ThroughHole:R_Axial_DIN0207_L6.3mm_D2.5mm_P7.62mm_Horizontal, symbol device:R
- added J1: Audio-Jack-3_2Switches, Connectors:PJ320E_3.5mm_Jack, symbol conn:Audio-Jack-3_2Switches
- BD2: renamed from D2B; footprint Diodes_SMD:D_0805 -> SoftEggKiCAD:D_DO-35_SOD27_P7.62mm_Horizontal+SMD
- C1: footprint Capacitors_SMD:C_0805_HandSoldering -> SoftEggKiCAD:C_Disc_D5.0mm_W2.5mm_P5.00mm+SMD
- D1: footprint Diodes_ThroughHole:D_DO-35_SOD27_P7.62mm_Horizontal -> SoftEggKiCAD:D_DO-35_SOD27_P7.62mm_Horizontal+SMD
- LS1: footprint Pin_Headers:Pin_Header_Angled_1x02_Pitch1.27mm -> Pin_Headers:Pin_Header_Straight_1x02_Pitch2.54mm
- R1, R2: footprint Resistors_SMD:R_0805_HandSoldering -> SoftEggKiCAD:R_Axial_DIN0204_L3.6mm_D1.6mm_P7.62mm_Horizontal+SMD804
- SW1: footprint Buttons_Switches_SMD:SW_SPST_EVQP0 -> SVTmaker:MSS22D18
- U1: footprint myelin-kicad:stm32f103c8t6-module-china -> SoftEggKiCAD:stm32f103c8t6-module-china-smd
Connections:
- wire segments 60 -> 62
Other:
- moved on the sheet: LS1
Changed lines of the file:
@@
 EESchema Schematic File Version 4
 LIBS:Stylish-Belt-Synth - Full-cache
-EELAYER 26 0
+EELAYER 28 0
 EELAYER END
 $Descr A4 11693 8268
@@
 Sheet 1 3
 Title "\"Stylish\" Trucker Belt Stylus Synthesizer"
-Date "2018-02-19"
-Rev "0.1"
+Date "2018-10-14"
+Rev "0.2"
 Comp "SoftEgg"
 Comment1 "V0.1 T.B. Trzepacz 2018/2/19"
-Comment2 ""
+Comment2 "V0.2 T.B. Trzepacz 2018/10/14"
 Comment3 ""
 Comment4 ""
@@
 F 0 "U1" H 5250 4750 60  0000 C CNN
 F 1 "stm32f103c8t6-module-china" V 5250 3400 60  0000 C CNN
-F 2 "myelin-kicad:stm32f103c8t6-module-china" H 5250 1700 60  0001 C CNN
+F 2 "SoftEggKiCAD:stm32f103c8t6-module-china-smd" H 5250 1700 60  0001 C CNN
 F 3 "" H 4850 3650 60  0000 C CNN
 	1    5250 3400
@@
 F 0 "R2" V 8930 5925 50  0000 C CNN
 F 1 "1k" V 8850 5925 50  0000 C CNN
-F 2 "Resistors_SMD:R_0805_HandSoldering" V 8780 5925 50  0001 C CNN
+F 2 "SoftEggKiCAD:R_Axial_DIN0204_L3.6mm_D1.6mm_P7.62mm_Horizontal+SMD804" V 8780 5925 50  0001 C CNN
 F 3 "" H 8850 5925 50  0001 C CNN
 	1    8850 5925
@@
 F 0 "C1" V 8350 5850 50  0000 L CNN
 F 1 "1uF" H 8460 5795 50  0001 L CNN
-F 2 "Capacitors_SMD:C_0805_HandSoldering" H 8450 5875 50  0001 C CNN
+F 2 "SoftEggKiCAD:C_Disc_D5.0mm_W2.5mm_P5.00mm+SMD" H 8450 5875 50  0001 C CNN
 F 3 "" H 8450 5875 50  0001 C CNN
 	1    8450 5875
@@
 F 0 "R1" V 8280 6075 50  0000 C CNN
 F 1 "10k" V 8200 6075 50  0000 C CNN
-F 2 "Resistors_SMD:R_0805_HandSoldering" V 8130 6075 50  0001 C CNN
+F 2 "SoftEggKiCAD:R_Axial_DIN0204_L3.6mm_D1.6mm_P7.62mm_Horizontal+SMD804" V 8130 6075 50  0001 C CNN
 F 3 "" H 8200 6075 50  0001 C CNN
 	1    8200 6075
@@
 L device:Speaker LS1
 U 1 1 5A8BCD0B
-P 9950 4900
-F 0 "LS1" H 10000 5125 50  0000 R CNN
-F 1 "Speaker" H 10000 5050 50  0000 R CNN
-F 2 "Pin_Headers:Pin_Header_Angled_1x02_Pitch1.27mm" H 9950 4700 50  0001 C CNN
-F 3 "" H 9940 4850 50  0001 C CNN
-	1    9950 4900
+P 10775 4875
+F 0 "LS1" H 10825 4675 50  0000 R CNN
+F 1 "Speaker" H 10900 5075 50  0000 R CNN
+F 2 "Pin_Headers:Pin_Header_Straight_1x02_Pitch2.54mm" H 10775 4675 50  0001 C CNN
+F 3 "" H 10765 4825 50  0001 C CNN
+	1    10775 4875
 	1    0    0    -1
 $EndComp
@@
 F 0 "SW1" H 2050 5750 50  0000 C CNN
 F 1 "Power" H 2175 5575 50  0000 C CNN
-F 2 "Buttons_Switches_SMD:SW_SPST_EVQP0" H 2175 5675 50  0001 C CNN
+F 2 "SVTmaker:MSS22D18" H 2175 5675 50  0001 C CNN
 F 3 "" H 2175 5675 50  0001 C CNN
 	1    2175 5675
@@
 $EndSheet
 Wire Wire Line
-	9750 4900 9150 4900
-Wire Wire Line
 	9150 5000 9750 5000
 Wire Wire Line
@@
 	1650 5675 1800 5675
 Connection ~ 1800 5675
-$Comp
-L device:R R1B
-U 1 1 5B95BBFA
-P 8200 5975
-F 0 "R1B" V 8280 5975 50  0001 C CNN
-F 1 "10k" V 8200 5975 50  0000 C CNN
-F 2 "Resistors_ThroughHole:R_Axial_DIN0204_L3.6mm_D1.6mm_P7.62mm_Horizontal" V 8130 5975 50  0001 C CNN
-F 3 "" H 8200 5975 50  0001 C CNN
-	1    8200 5975
-	0    1    1    0
-$EndComp
 Wire Notes Line
 	7525 5525 10650 5525
 Wire Notes Line
 	10650 5525 10650 6200
-$Comp
-L device:C_Small C1B
-U 1 1 5B9899BC
-P 8600 5875
-F 0 "C1B" V 8700 5775 50  0001 L CNN
-F 1 "1uF" H 8610 5795 50  0001 L CNN
-F 2 "Capacitors_ThroughHole:C_Disc_D5.0mm_W2.5mm_P5.00mm" H 8600 5875 50  0001 C CNN
-F 3 "" H 8600 5875 50  0001 C CNN
-	1    8600 5875
-	1    0    0    -1
-$EndComp
-$Comp
-L device:R R2B
-U 1 1 5B989A42
-P 9025 5925
-F 0 "R2B" V 9105 5925 50  0001 C CNN
-F 1 "1k" V 9025 5925 50  0000 C CNN
-F 2 "Resistors_ThroughHole:R_Axial_DIN0207_L6.3mm_D2.5mm_P7.62mm_Horizontal" V 8955 5925 50  0001 C CNN
-F 3 "" H 9025 5925 50  0001 C CNN
-	1    9025 5925
-	1    0    0    -1
-$EndComp
-Wire Wire Line
-	8050 5975 8050 6075
-Connection ~ 8050 6075
-Wire Wire Line
-	8350 5975 8350 6075
-Connection ~ 8350 6075
-Wire Wire Line
-	8600 5975 8450 5975
-Connection ~ 8450 5975
-Wire Wire Line
-	8600 5775 8450 5775
-Connection ~ 8450 5775
-Wire Wire Line
-	9025 5775 8850 5775
-Connection ~ 8850 5775
-Wire Wire Line
-	9025 6075 8850 6075
-Connection ~ 8850 6075
 Text Notes 9150 5825 0    50   ~ 0
 Doubled parts for thru-hole vs SMD
@@
 F 0 "D1" V 8250 3350 50  0000 R CNN
 F 1 "1N4148" V 8150 3550 50  0000 R CNN
-F 2 "Diodes_ThroughHole:D_DO-35_SOD27_P7.62mm_Horizontal" H 8200 3025 50  0001 C CNN
+F 2 "SoftEggKiCAD:D_DO-35_SOD27_P7.62mm_Horizontal+SMD" H 8200 3025 50  0001 C CNN
 F 3 "http://www.nxp.com/documents/data_sheet/1N4148_1N4448.pdf" H 8200 3200 50  0001 C CNN
 	1    8200 3200
@@
 	8200 2850 8200 3050
 Wire Wire Line
-	8800 3350 8875 3350
-Connection ~ 8800 3350
-$Comp
-L diode:1N4148 D2
-U 1 1 5BBC37C5
-P 8800 3200
-F 0 "D2" V 8846 3121 50  0000 R CNN
-F 1 "1N4148" V 8755 3121 50  0000 R CNN
-F 2 "Diodes_ThroughHole:D_DO-35_SOD27_P7.62mm_Horizontal" H 8800 3025 50  0001 C CNN
-F 3 "http://www.nxp.com/documents/data_sheet/1N4148_1N4448.pdf" H 8800 3200 50  0001 C CNN
-	1    8800 3200
-	0    -1   -1   0
-$EndComp
-Wire Wire Line
-	8875 3025 8800 3025
-Wire Wire Line
-	8800 3025 8800 3050
-Wire Wire Line
-	8800 3025 8675 3025
-Connection ~ 8800 3025
-Wire Wire Line
 	8200 2850 8025 2850
 Connection ~ 8200 2850
@@
 	8875 2675 8025 2675
 $Comp
-L diode:1N4148 D1B
-U 1 1 5BBE4231
-P 8325 3200
-F 0 "D1B" V 8375 3350 50  0001 R CNN
-F 1 "1N4148" V 8275 3550 50  0001 R CNN
-F 2 "Diodes_SMD:D_0805" H 8325 3025 50  0001 C CNN
-F 3 "http://www.nxp.com/documents/data_sheet/1N4148_1N4448.pdf" H 8325 3200 50  0001 C CNN
-	1    8325 3200
-	0    -1   -1   0
-$EndComp
-Wire Wire Line
-	8325 3050 8200 3050
-Connection ~ 8200 3050
-Wire Wire Line
-	8200 3350 8325 3350
-Connection ~ 8325 3350
-$Comp
-L diode:1N4148 D2B
+L diode:1N4148 BD2
 U 1 1 5BBE6FB8
 P 8675 3200
-F 0 "D2B" V 8721 3121 50  0001 R CNN
+F 0 "BD2" V 8721 3121 50  0001 R CNN
 F 1 "1N4148" V 8675 3121 50  0001 R CNN
-F 2 "Diodes_SMD:D_0805" H 8675 3025 50  0001 C CNN
+F 2 "SoftEggKiCAD:D_DO-35_SOD27_P7.62mm_Horizontal+SMD" H 8675 3025 50  0001 C CNN
 F 3 "http://www.nxp.com/documents/data_sheet/1N4148_1N4448.pdf" H 8675 3200 50  0001 C CNN
 	1    8675 3200
@@
 Wire Wire Line
 	8675 3025 8025 3025
-Wire Wire Line
-	8675 3350 8800 3350
 Connection ~ 8675 3350
-Wire Wire Line
-	8325 3350 8675 3350
 $Comp
 L conn:USB_B J0
@@
 	2725 2750 3275 2750
 $Comp
-L power:GND #PWR?
+L power:GND #PWR0107
 U 1 1 5BBEFFF4
 P 3275 2750
-F 0 "#PWR?" H 3275 2500 50  0001 C CNN
+F 0 "#PWR0107" H 3275 2500 50  0001 C CNN
 F 1 "GND" H 3280 2577 50  0000 C CNN
 F 2 "" H 3275 2750 50  0001 C CNN
@@
 Wire Wire Line
 	3250 4550 4200 4550
+$Comp
+L conn:Audio-Jack-3_2Switches J1
+U 1 1 5BC093A8
+P 10100 4900
+F 0 "J1" H 9813 4970 50  0000 R CNN
+F 1 "Audio-Jack-3_2Switches" H 10400 4625 50  0000 R CNN
+F 2 "Connectors:PJ320E_3.5mm_Jack" H 10350 5000 50  0001 C CNN
+F 3 "~" H 10350 5000 50  0001 C CNN
+	1    10100 4900
+	-1   0    0    -1
+$EndComp
+Wire Wire Line
+	9750 5000 9750 5100
+Wire Wire Line
+	9750 5100 10300 5100
+Wire Wire Line
+	9150 4900 9875 4900
+Wire Wire Line
+	9900 4800 9875 4800
+Wire Wire Line
+	9875 4800 9875 4900
+Connection ~ 9875 4900
+Wire Wire Line
+	9875 4900 9900 4900
+Wire Wire Line
+	10300 5100 10575 5100
+Wire Wire Line
+	10575 5100 10575 4975
+Connection ~ 10300 5100
+Wire Wire Line
+	9900 4700 9900 4550
+Wire Wire Line
+	9900 4550 10575 4550
+Wire Wire Line
+	10575 4550 10575 4875
+Wire Wire Line
+	9900 5000 9800 5000
+Wire Wire Line
+	9800 5000 9800 4550
+Wire Wire Line
+	9800 4550 9900 4550
+Connection ~ 9900 4550
+Wire Wire Line
+	8200 3350 8675 3350
+Wire Wire Line
+	8675 3350 8875 3350
+Wire Wire Line
+	8675 3025 8875 3025
 $EndSCHEMATC

Commit message: Updated footprints. Including STL for speaker holder.
Parts:
- added D3, D4: 1N5822, SoftEggKiCAD:D_DO-35_SOD27_P7.62mm_Horizontal+SMD, symbol device:D_Schottky
- C1: value 1uF -> 1μF
- J1: footprint Connectors:PJ320E_3.5mm_Jack -> Connectors:Stereo_Jack_3.5mm_Switch_Ledino_KB3SPRS
- R1: value 10k -> 10kΩ
- renumbered BD2 to D2
Connections:
- wire segments 62 -> 64
Changed lines of the file:
@@
 P 8450 5875
 F 0 "C1" V 8350 5850 50  0000 L CNN
-F 1 "1uF" H 8460 5795 50  0001 L CNN
+F 1 "1μF" H 8460 5795 50  0000 L CNN
 F 2 "SoftEggKiCAD:C_Disc_D5.0mm_W2.5mm_P5.00mm+SMD" H 8450 5875 50  0001 C CNN
 F 3 "" H 8450 5875 50  0001 C CNN
@@
 P 8200 6075
 F 0 "R1" V 8280 6075 50  0000 C CNN
-F 1 "10k" V 8200 6075 50  0000 C CNN
+F 1 "10kΩ" V 8200 6075 50  0000 C CNN
 F 2 "SoftEggKiCAD:R_Axial_DIN0204_L3.6mm_D1.6mm_P7.62mm_Horizontal+SMD804" V 8130 6075 50  0001 C CNN
 F 3 "" H 8200 6075 50  0001 C CNN
@@
 L conn:Conn_01x02 BT2
 U 1 1 5B9344BC
-P 1450 5925
-F 0 "BT2" H 1370 5692 50  0000 C CNN
-F 1 "Conn_01x02" H 1370 5691 50  0001 C CNN
-F 2 "Pin_Headers:Pin_Header_Angled_1x02_Pitch2.54mm" H 1450 5925 50  0001 C CNN
-F 3 "~" H 1450 5925 50  0001 C CNN
-	1    1450 5925
-	-1   0    0    1
-$EndComp
-Wire Wire Line
-	1650 5925 1650 6075
+P 1450 5825
+F 0 "BT2" H 1370 5592 50  0000 C CNN
+F 1 "Conn_01x02" H 1370 5591 50  0001 C CNN
+F 2 "Pin_Headers:Pin_Header_Angled_1x02_Pitch2.54mm" H 1450 5825 50  0001 C CNN
+F 3 "~" H 1450 5825 50  0001 C CNN
+	1    1450 5825
+	-1   0    0    -1
+$EndComp
 Wire Wire Line
 	1650 6075 1800 6075
@@
 Text Label 9200 5100 0    50   ~ 0
 +5V
-Text Label 2550 5675 0    50   ~ 0
+Text Label 3050 5675 0    50   ~ 0
 +5V
 Text Label 4200 4550 2    50   ~ 0
@@
 Connection ~ 4200 4700
 Wire Wire Line
-	1800 6075 2575 6075
+	1800 6075 3075 6075
 Connection ~ 1800 6075
 $Comp
 L power:GND #PWR0102
 U 1 1 5BACA4F7
-P 2575 6075
-F 0 "#PWR0102" H 2575 5825 50  0001 C CNN
-F 1 "GND" H 2580 5902 50  0000 C CNN
-F 2 "" H 2575 6075 50  0001 C CNN
-F 3 "" H 2575 6075 50  0001 C CNN
-	1    2575 6075
+P 3075 6075
+F 0 "#PWR0102" H 3075 5825 50  0001 C CNN
+F 1 "GND" H 3080 5902 50  0000 C CNN
+F 2 "" H 3075 6075 50  0001 C CNN
+F 3 "" H 3075 6075 50  0001 C CNN
+	1    3075 6075
 	1    0    0    -1
 $EndComp
@@
 	8875 2675 8025 2675
 $Comp
-L diode:1N4148 BD2
+L diode:1N4148 D2
 U 1 1 5BBE6FB8
 P 8675 3200
-F 0 "BD2" V 8721 3121 50  0001 R CNN
-F 1 "1N4148" V 8675 3121 50  0001 R CNN
+F 0 "D2" V 8721 3121 50  0000 R CNN
+F 1 "1N4148" V 8625 3125 50  0000 R CNN
 F 2 "SoftEggKiCAD:D_DO-35_SOD27_P7.62mm_Horizontal+SMD" H 8675 3025 50  0001 C CNN
 F 3 "http://www.nxp.com/documents/data_sheet/1N4148_1N4448.pdf" H 8675 3200 50  0001 C CNN
@@
 Wire Wire Line
 	3250 3350 3250 4550
-Wire Wire Line
-	3250 4550 4200 4550
 $Comp
 L conn:Audio-Jack-3_2Switches J1
@@
 F 0 "J1" H 9813 4970 50  0000 R CNN
 F 1 "Audio-Jack-3_2Switches" H 10400 4625 50  0000 R CNN
-F 2 "Connectors:PJ320E_3.5mm_Jack" H 10350 5000 50  0001 C CNN
+F 2 "Connectors:Stereo_Jack_3.5mm_Switch_Ledino_KB3SPRS" H 10350 5000 50  0001 C CNN
 F 3 "~" H 10350 5000 50  0001 C CNN
 	1    10100 4900
@@
 Wire Wire Line
 	8675 3025 8875 3025
+$Comp
+L device:D_Schottky D3
+U 1 1 5BC7018F
+P 2700 5675
+F 0 "D3" H 2700 5459 50  0000 C CNN
+F 1 "1N5822" H 2700 5550 50  0000 C CNN
+F 2 "SoftEggKiCAD:D_DO-35_SOD27_P7.62mm_Horizontal+SMD" H 2700 5675 50  0001 C CNN
+F 3 "~" H 2700 5675 50  0001 C CNN
+	1    2700 5675
+	-1   0    0    1
+$EndComp
+Wire Wire Line
+	2850 5675 3050 5675
+$Comp
+L device:D_Schottky D4
+U 1 1 5BC81B93
+P 3625 4550
+F 0 "D4" H 3625 4334 50  0000 C CNN
+F 1 "1N5822" H 3625 4425 50  0000 C CNN
+F 2 "SoftEggKiCAD:D_DO-35_SOD27_P7.62mm_Horizontal+SMD" H 3625 4550 50  0001 C CNN
+F 3 "~" H 3625 4550 50  0001 C CNN
+	1    3625 4550
+	-1   0    0    1
+$EndComp
+Wire Wire Line
+	3250 4550 3475 4550
+Wire Wire Line
+	3775 4550 4200 4550
+Wire Wire Line
+	1650 5925 1650 6075
 $EndSCHEMATC
