File: MAG Synth/Stylish-Belt-Synth - Full.sch (KiCad schematic (older format))
At the start: 20 parts, among them J0 USB_B, J1 Audio-Jack-3_2Switches, J26 WRITE PATCH, J27 PARAM SELECT, J28 PATCH SELECT, J29 MODE, J30 STYLUS, SW1 Power, U1 stm32f103c8t6-module-china

Commit message: V0.2 PCB completed! Schematic, PCB, and Gerbers updated.
Parts:
- BT1, BT2: footprint Pin_Headers:Pin_Header_Angled_1x02_Pitch2.54mm -> Pin_Headers:Pin_Header_Straight_1x02_Pitch2.54mm
- SW1: footprint SVTmaker:MSS22D18 -> SoftEggKiCAD:MSS22D18+THT; symbol switches:SW_SPST -> SoftEggKicadLib:SW_DPDT
Other:
- moved on the sheet: BT1, D3
Changed lines of the file:
@@
-$EndComp
-$Comp
-L device:Battery BT1
-U 1 1 5A85ADEB
-P 1800 5875
-F 0 "BT1" H 1900 5925 50  0000 L CNN
-F 1 "4 x 1.5V" H 1900 5800 50  0000 L CNN
-F 2 "Pin_Headers:Pin_Header_Angled_1x02_Pitch2.54mm" V 1800 5935 50  0001 C CNN
-F 3 "" V 1800 5935 50  0001 C CNN
-	1    1800 5875
-	1    0    0    -1
 $EndComp
 $Comp
@@
 	8850 5775 8850 5625
 $Comp
-L switches:SW_SPST SW1
+L SoftEggKicadLib:SW_DPDT SW1
 U 1 1 5A8C1199
-P 2175 5675
-F 0 "SW1" H 2050 5750 50  0000 C CNN
-F 1 "Power" H 2175 5575 50  0000 C CNN
-F 2 "SVTmaker:MSS22D18" H 2175 5675 50  0001 C CNN
-F 3 "" H 2175 5675 50  0001 C CNN
-	1    2175 5675
-	1    0    0    -1
-$EndComp
-Wire Wire Line
-	2550 5675 2375 5675
+P 2475 5875
+F 0 "SW1" H 2350 5950 50  0000 C CNN
+F 1 "Power" H 2475 5500 50  0000 C CNN
+F 2 "SoftEggKiCAD:MSS22D18+THT" H 2475 5875 50  0001 C CNN
+F 3 "" H 2475 5875 50  0001 C CNN
+	1    2475 5875
+	1    0    0    -1
+$EndComp
+Wire Wire Line
+	2850 5575 2675 5575
 Text Notes 9150 6125 0    60   ~ 0
 R/C Circuit to convert \nPWM pulses to waveform
@@
 Text Notes 4825 1825 0    60   ~ 0
 STM32F103C8T6\n"Blue Pill" board
-Wire Wire Line
-	1800 5675 1975 5675
 Wire Wire Line
 	8450 6075 8850 6075
@@
 L conn:Conn_01x02 BT2
 U 1 1 5B9344BC
-P 1450 5825
-F 0 "BT2" H 1370 5592 50  0000 C CNN
-F 1 "Conn_01x02" H 1370 5591 50  0001 C CNN
-F 2 "Pin_Headers:Pin_Header_Angled_1x02_Pitch2.54mm" H 1450 5825 50  0001 C CNN
-F 3 "~" H 1450 5825 50  0001 C CNN
-	1    1450 5825
-	-1   0    0    -1
-$EndComp
-Wire Wire Line
-	1650 6075 1800 6075
-Wire Wire Line
-	1650 5825 1650 5675
-Wire Wire Line
-	1650 5675 1800 5675
-Connection ~ 1800 5675
+P 1275 5475
+F 0 "BT2" H 1195 5242 50  0000 C CNN
+F 1 "Conn_01x02" H 1195 5241 50  0001 C CNN
+F 2 "Pin_Headers:Pin_Header_Straight_1x02_Pitch2.54mm" H 1275 5475 50  0001 C CNN
+F 3 "~" H 1275 5475 50  0001 C CNN
+	1    1275 5475
+	0    1    -1   0
+$EndComp
 Wire Notes Line
 	7525 5525 10650 5525
@@
 Text Label 9200 5100 0    50   ~ 0
 +5V
-Text Label 3050 5675 0    50   ~ 0
+Text Label 3350 5575 0    50   ~ 0
 +5V
 Text Label 4200 4550 2    50   ~ 0
@@
 	4200 4700 3950 4700
 Connection ~ 4200 4700
-Wire Wire Line
-	1800 6075 3075 6075
-Connection ~ 1800 6075
 $Comp
 L power:GND #PWR0102
 U 1 1 5BACA4F7
-P 3075 6075
-F 0 "#PWR0102" H 3075 5825 50  0001 C CNN
-F 1 "GND" H 3080 5902 50  0000 C CNN
-F 2 "" H 3075 6075 50  0001 C CNN
-F 3 "" H 3075 6075 50  0001 C CNN
-	1    3075 6075
+P 3350 6100
+F 0 "#PWR0102" H 3350 5850 50  0001 C CNN
+F 1 "GND" H 3355 5927 50  0000 C CNN
+F 2 "" H 3350 6100 50  0001 C CNN
+F 3 "" H 3350 6100 50  0001 C CNN
+	1    3350 6100
 	1    0    0    -1
 $EndComp
@@
 L device:D_Schottky D3
 U 1 1 5BC7018F
-P 2700 5675
-F 0 "D3" H 2700 5459 50  0000 C CNN
-F 1 "1N5822" H 2700 5550 50  0000 C CNN
-F 2 "SoftEggKiCAD:D_DO-35_SOD27_P7.62mm_Horizontal+SMD" H 2700 5675 50  0001 C CNN
-F 3 "~" H 2700 5675 50  0001 C CNN
-	1    2700 5675
+P 3000 5575
+F 0 "D3" H 3000 5359 50  0000 C CNN
+F 1 "1N5822" H 3000 5450 50  0000 C CNN
+F 2 "SoftEggKiCAD:D_DO-35_SOD27_P7.62mm_Horizontal+SMD" H 3000 5575 50  0001 C CNN
+F 3 "~" H 3000 5575 50  0001 C CNN
+	1    3000 5575
 	-1   0    0    1
 $EndComp
 Wire Wire Line
-	2850 5675 3050 5675
+	3150 5575 3350 5575
 $Comp
 L device:D_Schottky D4
@@
 	3775 4550 4200 4550
 Wire Wire Line
-	1650 5925 1650 6075
+	2675 5925 3350 5925
+Wire Wire Line
+	3350 5925 3350 6100
+Wire Wire Line
+	1800 5675 2275 5675
+$Comp
+L device:Battery BT1
+U 1 1 5A85ADEB
+P 1600 5675
+F 0 "BT1" V 1475 5600 50  0000 L CNN
+F 1 "4 x 1.5V" V 1725 5525 50  0000 L CNN
+F 2 "Pin_Headers:Pin_Header_Straight_1x02_Pitch2.54mm" V 1600 5735 50  0001 C CNN
+F 3 "" V 1600 5735 50  0001 C CNN
+	1    1600 5675
+	0    1    1    0
+$EndComp
+Wire Wire Line
+	1400 5675 1275 5675
+Wire Wire Line
+	2275 6025 1175 6025
+Wire Wire Line
+	1175 6025 1175 5675
 $EndSCHEMATC

Commit message: V3 board V2.4 case
Parts:
- removed BT1: 4 x 1.5V, Pin_Headers:Pin_Header_Straight_1x02_Pitch2.54mm, symbol device:Battery
- removed BT2: Conn_01x02, Pin_Headers:Pin_Header_Straight_1x02_Pitch2.54mm, symbol conn:Conn_01x02
- added BT12, BT34: ~, SoftEggKiCAD:AA_Battery_Dual_Terminal, symbol SoftEggKicadLib:AABatteryEnd
- added BTN1, BTN3: -, SoftEggKiCAD:AA_Battery_-_Terminal, symbol conn:Conn_01x01
- added BTP2, BTP4: +, SoftEggKiCAD:AA_Battery_+_Terminal, symbol conn:Conn_01x01
- added C2: 1000μF, Capacitors_ThroughHole:CP_Radial_D10.0mm_P5.00mm, symbol device:CP
- added C3: 470μF, Capacitors_ThroughHole:CP_Radial_D10.0mm_P5.00mm, symbol device:CP
- added CA1: 470μF, SoftEggKiCAD:C_Disc_D5.0mm_W2.5mm_P5.00mm+SMD, symbol device:C_Small
- added CA2: 1μF, SoftEggKiCAD:C_Disc_D5.0mm_W2.5mm_P5.00mm+SMD, symbol device:C_Small
- added CA3: 1μF, Capacitors_ThroughHole:CP_Radial_Tantal_D4.5mm_P2.50mm, symbol device:C_Small
- added CA4: 0.39μF, SoftEggKiCAD:C_Disc_D5.0mm_W2.5mm_P5.00mm+SMD, symbol device:C_Small
- added R3: 120Ω, SoftEggKiCAD:R_Axial_DIN0204_L3.6mm_D1.6mm_P7.62mm_Horizontal+SMD804, symbol device:R
- added RA1: 100Ω, SoftEggKiCAD:R_Axial_DIN0204_L3.6mm_D1.6mm_P7.62mm_Horizontal+SMD804, symbol device:R
- added RV1: Volume, SoftEggKiCAD:Wheel_Pot_W_Switch_RV12_B103_FUSTAR, symbol SoftEggKicadLib:Switch_Pot
- added U2: XPT8871, SMD_Packages:SOIC-8-N, symbol SoftEggKicadLib:XPT8871
- J1: value Audio-Jack-3_2Switches -> Headphone
- R1: value 10kΩ -> 8Ω
- R2: value 1k -> 47Ω
- SW1: value Power -> OVERDRIVE
Connections:
- net labels added: +3.3V, VUSB
- net labels removed: PWM_Audio_Out
- wire segments 64 -> 97
Other:
- note added: "Amplifier Stage"
- note added: "Diode isolates \nUSB power \nfrom battery power."
- note added: "Diodes create 4th button input\nas 2nd and 3rd button simultaneous press."
- note added: "Headphone jack \ndetaches speaker.\nJumper 1,2,5,4 \nif no headphone jack."
- note added: "Keyboard is pattern \non front of PCB."
- note added: "Next revision we try\nmounting battery clips to the PCB.\n"
- note added: "PWM Output Filter"
- note added: "Power Input"
- note added: "Power filtering\ncapacitors might\nbe optional."
- note added: "Stylus is\nattached via\nbanana plug."
- note added: "Switch is ganged with \nwheel potentiometer."
- note removed: "Battery clip glued\n to back of board"
- note removed: "Doubled parts for thru-hole vs SMD"
- note removed: "Use only one set of parts"
- moved on the sheet: C1, D1, D2, D3, D4, J1, J26, J27, J28, J29, J30, LS1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

Commit message: More board cleanup. Fixed values of parts based on test board construction. Rewired potentiometer so that low volume is nearest the power on/off click. More hand vias where they are needed.
Parts:
- added BT12H1, BT34H1: Battery, Battery_Holders:BatteryHolder_Keystone_2462_2xAA, symbol device:Battery
- R2: value 47Ω -> 47KΩ
- R3: value 120Ω -> 44Ω
- SW1: footprint SoftEggKiCAD:MSS22D18+THT -> Pin_Headers:Pin_Header_Straight_1x03_Pitch2.54mm; symbol SoftEggKicadLib:SW_DPDT -> switches:SW_SPDT
Connections:
- wire segments 97 -> 103
Other:
- note removed: "Next revision we try\nmounting battery clips to the PCB.\n"
- moved on the sheet: RV1
Changed lines of the file:
@@
 F 3 "~" H 9750 3325 50  0001 C CNN
 	1    9750 3325
-	0    -1   1    0
+	0    1    1    0
 $EndComp
 Connection ~ 9075 6000
@@
 Text Notes 11000 2172 2    47   ~ 0
 Power filtering\ncapacitors might\nbe optional.
-Text Notes 8175 2150 0    47   ~ 0
-Next revision we try\nmounting battery clips to the PCB.\n
 Text Notes 10000 3050 0    47   ~ 0
 Switch is ganged with \nwheel potentiometer.
@@
 Keyboard is pattern \non front of PCB.
 Wire Wire Line
-	9575 2875 9600 2875
-Wire Wire Line
-	9900 2875 10300 2875
-Connection ~ 10300 2875
-Wire Wire Line
 	10300 2875 10875 2875
 $Comp
@@
 Wire Wire Line
 	9575 1950 9575 2425
-Connection ~ 9575 2425
-Wire Wire Line
-	9575 2425 9575 2875
 Wire Wire Line
 	9750 3475 9750 3775
@@
 P 8825 3550
 F 0 "R2" H 8700 3700 50  0000 L CNN
-F 1 "47Ω" V 8825 3475 50  0000 L CNN
+F 1 "47KΩ" V 8825 3475 39  0000 L CNN
 F 2 "SoftEggKiCAD:R_Axial_DIN0204_L3.6mm_D1.6mm_P7.62mm_Horizontal+SMD804" V 8755 3550 50  0001 C CNN
 F 3 "~" H 8825 3550 50  0001 C CNN
@@
 P 4450 6150
 F 0 "R3" V 4350 6150 50  0000 C CNN
-F 1 "120Ω" V 4450 6150 50  0000 C CNN
+F 1 "44Ω" V 4450 6150 50  0000 C CNN
 F 2 "SoftEggKiCAD:R_Axial_DIN0204_L3.6mm_D1.6mm_P7.62mm_Horizontal+SMD804" V 4380 6150 50  0001 C CNN
 F 3 "~" H 4450 6150 50  0001 C CNN
@@
 Wire Wire Line
 	4600 6150 5000 6150
-$Comp
-L SoftEggKicadLib:SW_DPDT SW1
-U 1 1 5CE36C2E
-P 9300 3750
-F 0 "SW1" H 9225 3825 50  0000 R CNN
-F 1 "OVERDRIVE" H 9500 3350 50  0000 R CNN
-F 2 "SoftEggKiCAD:MSS22D18+THT" H 9300 3750 50  0001 C CNN
-F 3 "" H 9300 3750 50  0001 C CNN
-	1    9300 3750
-	1    0    0    -1
-$EndComp
 Wire Wire Line
 	8975 3800 8975 3550
@@
 	8975 3550 9100 3550
 Wire Wire Line
-	8825 3325 9550 3325
-Wire Wire Line
-	9500 3450 9550 3450
-Wire Wire Line
-	9550 3450 9550 3325
-Connection ~ 9550 3325
-Wire Wire Line
-	9550 3325 9600 3325
-Wire Wire Line
-	9500 3800 9550 3800
-Wire Wire Line
-	9550 3800 9550 3450
-Connection ~ 9550 3450
-Wire Wire Line
-	8975 3800 8975 3900
-Wire Wire Line
-	8975 3900 9100 3900
-Connection ~ 8975 3800
+	8825 3325 9525 3325
 $Comp
 L conn:Conn_01x01 BTN1
@@
 	8700 2425 8900 2425
 Wire Wire Line
-	9050 2425 9200 2425
+	9050 2425 9150 2425
 $Comp
 L SoftEggKicadLib:AABatteryEnd BT34
@@
 	0    -1   -1   0
 $EndComp
+$Comp
+L device:Battery BT34H1
+U 1 1 5D0F71F9
+P 8950 2300
+F 0 "BT34H1" V 8705 2300 50  0000 C CNN
+F 1 "Battery" V 8796 2300 50  0000 C CNN
+F 2 "Battery_Holders:BatteryHolder_Keystone_2462_2xAA" V 8950 2360 50  0001 C CNN
+F 3 "~" V 8950 2360 50  0001 C CNN
+	1    8950 2300
+	0    1    1    0
+$EndComp
+Wire Wire Line
+	8225 2425 8225 2300
+Wire Wire Line
+	8225 2300 8300 2300
+Connection ~ 8225 2425
+Wire Wire Line
+	8700 2425 8700 2300
+Wire Wire Line
+	8700 2300 8750 2300
+Connection ~ 8700 2300
+Wire Wire Line
+	9150 2300 9150 2425
+Connection ~ 9150 2425
+Wire Wire Line
+	9150 2425 9200 2425
+$Comp
+L device:Battery BT12H1
+U 1 1 5D0F49DB
+P 8500 2300
+F 0 "BT12H1" V 8255 2300 50  0000 C CNN
+F 1 "Battery" V 8346 2300 50  0000 C CNN
+F 2 "Battery_Holders:BatteryHolder_Keystone_2462_2xAA" V 8500 2360 50  0001 C CNN
+F 3 "~" V 8500 2360 50  0001 C CNN
+	1    8500 2300
+	0    1    1    0
+$EndComp
+Connection ~ 9525 3325
+Wire Wire Line
+	9525 3325 9600 3325
+Wire Wire Line
+	10300 2875 9950 2875
+Wire Wire Line
+	9950 2875 9950 2975
+Wire Wire Line
+	9950 2975 9600 2975
+Wire Wire Line
+	9600 2975 9600 2875
+Connection ~ 10300 2875
+Wire Wire Line
+	9900 2875 9900 2700
+Wire Wire Line
+	9900 2700 9575 2700
+Wire Wire Line
+	9575 2700 9575 2425
+Connection ~ 9575 2425
+$Comp
+L switches:SW_SPDT SW1
+U 1 1 5CE36C2E
+P 9300 3650
+F 0 "SW1" H 9400 3825 50  0000 R CNN
+F 1 "OVERDRIVE" H 9500 3425 50  0000 R CNN
+F 2 "Pin_Headers:Pin_Header_Straight_1x03_Pitch2.54mm" H 9300 3650 50  0001 C CNN
+F 3 "" H 9300 3650 50  0001 C CNN
+	1    9300 3650
+	-1   0    0    -1
+$EndComp
+Wire Wire Line
+	9525 3650 9525 3325
+Wire Wire Line
+	9500 3650 9525 3650
 $EndSCHEMATC

Commit message: PCB V4 update Wood CNC models added
Parts:
- removed SW1: OVERDRIVE, Pin_Headers:Pin_Header_Straight_1x03_Pitch2.54mm, symbol switches:SW_SPDT
- added C4: 4.7nF, SoftEggKiCAD:C_Disc_D5.0mm_W2.5mm_P5.00mm+SMD, symbol device:C_Small
- added CL16: 22µF, SoftEggKiCAD:C_Disc_D5.0mm_W2.5mm_P5.00mm+SMD, symbol device:CP1_Small
- added R4: 33kΩ, SoftEggKiCAD:R_Axial_DIN0204_L3.6mm_D1.6mm_P7.62mm_Horizontal+SMD804, symbol device:R
- C1: value 1μF -> 220nF
- R1: value 8Ω -> 330Ω
- R2: value 47KΩ -> 3.3kΩ
Connections:
- wire segments 103 -> 104
Other:
- note added: "This capacitor eliminates LED ring noise!"
- moved on the sheet: C1, R1, R2, R3
Changed lines of the file:
@@
 L device:C_Small C1
 U 1 1 5A8BA68B
-P 8825 4000
-F 0 "C1" V 8725 3975 50  0000 L CNN
-F 1 "1μF" H 8835 3920 50  0000 L CNN
-F 2 "SoftEggKiCAD:C_Disc_D5.0mm_W2.5mm_P5.00mm+SMD" H 8825 4000 50  0001 C CNN
-F 3 "" H 8825 4000 50  0001 C CNN
-	1    8825 4000
+P 8050 3550
+F 0 "C1" V 7950 3525 50  0000 L CNN
+F 1 "220nF" H 8060 3470 50  0000 L CNN
+F 2 "SoftEggKiCAD:C_Disc_D5.0mm_W2.5mm_P5.00mm+SMD" H 8050 3550 50  0001 C CNN
+F 3 "" H 8050 3550 50  0001 C CNN
+	1    8050 3550
 	1    0    0    -1
 $EndComp
@@
 L device:R R1
 U 1 1 5A8BA742
-P 8600 3800
-F 0 "R1" V 8680 3800 50  0000 C CNN
-F 1 "8Ω" V 8600 3800 50  0000 C CNN
-F 2 "SoftEggKiCAD:R_Axial_DIN0204_L3.6mm_D1.6mm_P7.62mm_Horizontal+SMD804" V 8530 3800 50  0001 C CNN
-F 3 "" H 8600 3800 50  0001 C CNN
-	1    8600 3800
+P 7875 3325
+F 0 "R1" V 7955 3325 50  0000 C CNN
+F 1 "330Ω" V 7875 3325 50  0000 C CNN
+F 2 "SoftEggKiCAD:R_Axial_DIN0204_L3.6mm_D1.6mm_P7.62mm_Horizontal+SMD804" V 7805 3325 50  0001 C CNN
+F 3 "" H 7875 3325 50  0001 C CNN
+	1    7875 3325
 	0    1    1    0
 $EndComp
@@
 R/C Circuit to convert \nPWM pulses to waveform
 Wire Notes Line
-	11075 4450 8325 4450
-Wire Notes Line
 	8350 575  11075 600
 Wire Notes Line
@@
 STM32F103C8T6\n"Blue Pill" board
 Wire Wire Line
-	8450 3800 8425 3800
-Text Label 8425 3800 1    50   ~ 0
+	7725 3325 7700 3325
+Text Label 7700 3325 3    50   ~ 0
 AUDIO_OUT
 Text Label 4050 4250 2    50   ~ 0
@@
 Wire Wire Line
 	5000 6050 4925 6050
-Wire Wire Line
-	4800 6250 5000 6250
 $Comp
 L SoftEggKicadLib:StylusKeyboardA KB1
@@
 Wire Wire Line
 	4200 4700 5500 4700
-Wire Notes Line
-	8325 3100 11075 3100
 Wire Notes Line
 	11075 3100 11075 4450
@@
 Text Label 4925 6050 2    50   ~ 0
 LED_DIN
-Text Label 4200 6150 2    50   ~ 0
+Text Label 3750 6150 2    50   ~ 0
 +3.3V
 Text Label 9075 6300 2    50   ~ 0
@@
 L power:GND #PWR0103
 U 1 1 5BACC962
-P 4800 6250
-F 0 "#PWR0103" H 4800 6000 50  0001 C CNN
-F 1 "GND" H 4805 6077 50  0000 C CNN
-F 2 "" H 4800 6250 50  0001 C CNN
-F 3 "" H 4800 6250 50  0001 C CNN
-	1    4800 6250
+P 4500 6400
+F 0 "#PWR0103" H 4500 6150 50  0001 C CNN
+F 1 "GND" H 4505 6227 50  0000 C CNN
+F 2 "" H 4500 6400 50  0001 C CNN
+F 3 "" H 4500 6400 50  0001 C CNN
+	1    4500 6400
 	1    0    0    -1
 $EndComp
@@
 L power:GND #PWR0106
 U 1 1 5BAD51F5
-P 8825 4175
-F 0 "#PWR0106" H 8825 3925 50  0001 C CNN
-F 1 "GND" H 8830 4002 50  0000 C CNN
-F 2 "" H 8825 4175 50  0001 C CNN
-F 3 "" H 8825 4175 50  0001 C CNN
-	1    8825 4175
-	1    0    0    -1
-$EndComp
-Text Label 10625 3775 0    50   ~ 0
+P 8050 3725
+F 0 "#PWR0106" H 8050 3475 50  0001 C CNN
+F 1 "GND" H 8055 3552 50  0000 C CNN
+F 2 "" H 8050 3725 50  0001 C CNN
+F 3 "" H 8050 3725 50  0001 C CNN
+	1    8050 3725
+	1    0    0    -1
+$EndComp
+Text Label 10625 3800 0    50   ~ 0
 PWM_OUT
-Wire Notes Line
-	8325 3100 8325 4450
 Wire Wire Line
 	6300 2000 6925 2000
@@
 	7825 5100 8025 5100
 Wire Wire Line
-	8750 3800 8825 3800
-Wire Wire Line
-	8825 4100 8825 4175
+	8050 3650 8050 3725
 Wire Wire Line
 	8550 2425 8225 2425
@@
 	8575 5100 8550 5100
 Wire Wire Line
-	8825 3800 8825 3900
-Wire Wire Line
 	9575 1950 9575 2425
 Wire Wire Line
-	9750 3475 9750 3775
-Wire Wire Line
-	9750 3775 10625 3775
+	9750 3475 9750 3800
+Wire Wire Line
+	9750 3800 10625 3800
 Wire Wire Line
 	9900 3325 10175 3325
@@
 Wire Wire Line
 	9775 5500 10275 5500
-$Comp
-L device:R R2
-U 1 1 5CE2A35E
-P 8825 3550
-F 0 "R2" H 8700 3700 50  0000 L CNN
-F 1 "47KΩ" V 8825 3475 39  0000 L CNN
-F 2 "SoftEggKiCAD:R_Axial_DIN0204_L3.6mm_D1.6mm_P7.62mm_Horizontal+SMD804" V 8755 3550 50  0001 C CNN
-F 3 "~" H 8825 3550 50  0001 C CNN
-	1    8825 3550
-	1    0    0    -1
-$EndComp
-Wire Wire Line
-	8825 3325 8825 3400
-Wire Wire Line
-	8825 3700 8825 3800
-Connection ~ 8825 3800
-Wire Wire Line
-	8825 3800 8975 3800
 Text Label 6300 2300 0    50   ~ 0
 +3.3V
-$Comp
-L device:R R3
-U 1 1 5CE50512
-P 4450 6150
-F 0 "R3" V 4350 6150 50  0000 C CNN
-F 1 "44Ω" V 4450 6150 50  0000 C CNN
-F 2 "SoftEggKiCAD:R_Axial_DIN0204_L3.6mm_D1.6mm_P7.62mm_Horizontal+SMD804" V 4380 6150 50  0001 C CNN
-F 3 "~" H 4450 6150 50  0001 C CNN
-	1    4450 6150
-	0    1    1    0
-$EndComp
-Wire Wire Line
-	4200 6150 4300 6150
-Wire Wire Line
-	4600 6150 5000 6150
-Wire Wire Line
-	8975 3800 8975 3550
-Wire Wire Line
-	8975 3550 9100 3550
-Wire Wire Line
-	8825 3325 9525 3325
+Wire Wire Line
+	3750 6150 3850 6150
 $Comp
 L conn:Conn_01x01 BTN1
@@
 	0    1    1    0
 $EndComp
-Connection ~ 9525 3325
-Wire Wire Line
-	9525 3325 9600 3325
 Wire Wire Line
 	10300 2875 9950 2875
@@
 Connection ~ 9575 2425
 $Comp
-L switches:SW_SPDT SW1
-U 1 1 5CE36C2E
-P 9300 3650
-F 0 "SW1" H 9400 3825 50  0000 R CNN
-F 1 "OVERDRIVE" H 9500 3425 50  0000 R CNN
-F 2 "Pin_Headers:Pin_Header_Straight_1x03_Pitch2.54mm" H 9300 3650 50  0001 C CNN
-F 3 "" H 9300 3650 50  0001 C CNN
-	1    9300 3650
-	-1   0    0    -1
-$EndComp
-Wire Wire Line
-	9525 3650 9525 3325
-Wire Wire Line
-	9500 3650 9525 3650
+L device:R R3
+U 1 1 5CE50512
+P 4000 6150
+F 0 "R3" V 3900 6150 50  0000 C CNN
+F 1 "44Ω" V 4000 6150 50  0000 C CNN
+F 2 "SoftEggKiCAD:R_Axial_DIN0204_L3.6mm_D1.6mm_P7.62mm_Horizontal+SMD804" V 3930 6150 50  0001 C CNN
+F 3 "~" H 4000 6150 50  0001 C CNN
+	1    4000 6150
+	0    1    1    0
+$EndComp
+Wire Wire Line
+	4500 6150 5000 6150
+$Comp
+L device:CP1_Small CL16
+U 1 1 5D1435CA
+P 4500 6250
+F 0 "CL16" V 4272 6250 50  0000 C CNN
+F 1 "22µF" V 4363 6250 50  0000 C CNN
+F 2 "SoftEggKiCAD:C_Disc_D5.0mm_W2.5mm_P5.00mm+SMD" H 4500 6250 50  0001 C CNN
+F 3 "~" H 4500 6250 50  0001 C CNN
+	1    4500 6250
+	1    0    0    -1
+$EndComp
+Wire Wire Line
+	4150 6150 4500 6150
+Connection ~ 4500 6150
+Wire Wire Line
+	5000 6250 4775 6250
+Wire Wire Line
+	4775 6250 4775 6350
+Wire Wire Line
+	4775 6350 4500 6350
+Wire Wire Line
+	4500 6350 4500 6400
+Connection ~ 4500 6350
+Text Notes 4200 6625 2    47   ~ 0
+This capacitor eliminates LED ring noise!
+Wire Notes Line style solid
+	4200 6550 4425 6300
+$Comp
+L device:R R2
+U 1 1 5CE2A35E
+P 8225 3325
+F 0 "R2" V 8300 3280 50  0000 L CNN
+F 1 "3.3kΩ" V 8225 3250 39  0000 L CNN
+F 2 "SoftEggKiCAD:R_Axial_DIN0204_L3.6mm_D1.6mm_P7.62mm_Horizontal+SMD804" V 8155 3325 50  0001 C CNN
+F 3 "~" H 8225 3325 50  0001 C CNN
+	1    8225 3325
+	0    1    1    0
+$EndComp
+Wire Wire Line
+	8050 3450 8050 3325
+Connection ~ 8050 3325
+Wire Wire Line
+	8050 3325 8075 3325
+Wire Wire Line
+	8025 3325 8050 3325
+$Comp
+L device:R R4
+U 1 1 5D1B92DC
+P 8575 3325
+F 0 "R4" V 8650 3280 50  0000 L CNN
+F 1 "33kΩ" V 8575 3250 39  0000 L CNN
+F 2 "SoftEggKiCAD:R_Axial_DIN0204_L3.6mm_D1.6mm_P7.62mm_Horizontal+SMD804" V 8505 3325 50  0001 C CNN
+F 3 "~" H 8575 3325 50  0001 C CNN
+	1    8575 3325
+	0    1    1    0
+$EndComp
+$Comp
+L device:C_Small C4
+U 1 1 5D1B9DA4
+P 8400 3550
+F 0 "C4" V 8300 3525 50  0000 L CNN
+F 1 "4.7nF" H 8410 3470 50  0000 L CNN
+F 2 "SoftEggKiCAD:C_Disc_D5.0mm_W2.5mm_P5.00mm+SMD" H 8400 3550 50  0001 C CNN
+F 3 "" H 8400 3550 50  0001 C CNN
+	1    8400 3550
+	1    0    0    -1
+$EndComp
+$Comp
+L power:GND #PWR?
+U 1 1 5D1B9DAF
+P 8400 3725
+F 0 "#PWR?" H 8400 3475 50  0001 C CNN
+F 1 "GND" H 8405 3552 50  0000 C CNN
+F 2 "" H 8400 3725 50  0001 C CNN
+F 3 "" H 8400 3725 50  0001 C CNN
+	1    8400 3725
+	1    0    0    -1
+$EndComp
+Wire Wire Line
+	8400 3450 8400 3325
+Wire Wire Line
+	8400 3650 8400 3725
+Wire Wire Line
+	8375 3325 8400 3325
+Wire Wire Line
+	8400 3325 8425 3325
+Connection ~ 8400 3325
+Wire Notes Line
+	7580 3100 11070 3100
+Wire Notes Line
+	7580 3100 7580 4450
+Wire Wire Line
+	8725 3325 9600 3325
+Wire Notes Line
+	11075 4450 7580 4450
 $EndSCHEMATC

Commit message: Small updates to PCB. One footprint changed so all SMD are 0805. BOM added. V1 of Source Code added.
Parts:
- CA1: value 470μF -> 220µF
Changed lines of the file:
@@
 AR Path="/5CD1D13D" Ref="CA1"  Part="1"
 F 0 "CA1" V 8375 5750 50  0000 L CNN
-F 1 "470μF" V 8375 5975 50  0000 L CNN
+F 1 "220µF" V 8375 5975 50  0000 L CNN
 F 2 "SoftEggKiCAD:C_Disc_D5.0mm_W2.5mm_P5.00mm+SMD" H 8450 5925 50  0001 C CNN
 F 3 "" H 8450 5925 50  0001 C CNN
